Commit message: Updated urdf

File: ros/catkin_ws/src/husky/husky_description/urdf/husky.urdf.xacro (robot description, xacro)
@@ -23,104 +23,19 @@
 <robot name="husky" xmlns:xacro="http://ros.org/wiki/xacro">
   <!-- IMU Link -->
-  <xacro:arg name="imu_xyz"     default="$(optenv HUSKY_IMU_XYZ 0.19 0 0.149)"/>
-  <xacro:arg name="imu_rpy"     default="$(optenv HUSKY_IMU_RPY 0 -1.5708 3.1416)"/>
-  <xacro:arg name="imu_parent"  default="$(optenv HUSKY_IMU_PARENT base_link)"/>
-  <!-- LMS1XX Laser Primary and Secondary -->
-  <xacro:arg name="laser_enabled"           default="$(optenv HUSKY_LMS1XX_ENABLED 0)" />
-  <xacro:arg name="laser_topic"             default="$(optenv HUSKY_LMS1XX_TOPIC front/scan)"/>
-  <xacro:arg name="laser_tower"             default="$(optenv HUSKY_LMS1XX_TOWER 1)"/>
-  <xacro:arg name="laser_prefix"            default="$(optenv HUSKY_LMS1XX_PREFIX front)"/>
-  <xacro:arg name="laser_parent"            default="$(optenv HUSKY_LMS1XX_PARENT top_plate_link)"/>
-  <xacro:arg name="laser_xyz"               default="$(optenv HUSKY_LMS1XX_XYZ 0.2206 0.0 0.00635)" />
-  <xacro:arg name="laser_rpy"               default="$(optenv HUSKY_LMS1XX_RPY 0.0 0.0 0.0)" />
-  <xacro:arg name="laser_secondary_enabled" default="$(optenv HUSKY_LMS1XX_SECONDARY_ENABLED 0)" />
-  <xacro:arg name="laser_secondary_topic"   default="$(optenv HUSKY_LMS1XX_SECONDARY_TOPIC rear/scan)"/>
-  <xacro:arg name="laser_secondary_tower"   default="$(optenv HUSKY_LMS1XX_SECONDARY_TOWER 1)"/>
-  <xacro:arg name="laser_secondary_prefix"  default="$(optenv HUSKY_LMS1XX_SECONDARY_PREFIX rear)"/>
-  <xacro:arg name="laser_secondary_parent"  default="$(optenv HUSKY_LMS1XX_SECONDARY_PARENT top_plate_link)"/>
-  <xacro:arg name="laser_secondary_xyz"     default="$(optenv HUSKY_LMS1XX_SECONDARY_XYZ -0.2206 0.0 0.00635)" />
-  <xacro:arg name="laser_secondary_rpy"     default="$(optenv HUSKY_LMS1XX_SECONDARY_RPY 0.0 0.0 3.14159)" />
-  <!-- UST10 Laser Primary  and Secondary -->
-  <xacro:arg name="laser_ust10_front_enabled" default="$(optenv HUSKY_UST10_ENABLED 0)" />
-  <xacro:arg name="laser_ust10_front_topic"   default="$(optenv HUSKY_UST10_TOPIC front/scan)" />
-  <xacro:arg name="laser_ust10_front_prefix"  default="$(optenv HUSKY_UST10_PREFIX front)" />
-  <xacro:arg name="laser_ust10_front_parent"  default="$(optenv HUSKY_UST10_PARENT top_plate_link)" />
-  <xacro:arg name="laser_ust10_front_xyz"     default="$(optenv HUSKY_UST10_XYZ 0.2206 0.0 0.00635)" />
-  <xacro:arg name="laser_ust10_front_rpy"     default="$(optenv HUSKY_UST10_RPY 0 0 0)" />
-  <xacro:arg name="laser_ust10_rear_enabled"  default="$(optenv HUSKY_UST10_SECONDARY_ENABLED 0)" />
-  <xacro:arg name="laser_ust10_rear_topic"    default="$(optenv HUSKY_UST10_SECONDARY_TOPIC rear/scan)" />
-  <xacro:arg name="laser_ust10_rear_prefix"   default="$(optenv HUSKY_UST10_SECONDARY_PREFIX rear)" />
-  <xacro:arg name="laser_ust10_rear_parent"   default="$(optenv HUSKY_UST10_SECONDARY_PARENT top_plate_link)" />
-  <xacro:arg name="laser_ust10_rear_xyz"      default="$(optenv HUSKY_UST10_SECONDARY_XYZ -0.2206 0.0 0.00635)" />
-  <xacro:arg name="laser_ust10_rear_rpy"      default="$(optenv HUSKY_UST10_SECONDARY_RPY 0 0 3.14159)" />
-  <!-- Velodyne LiDAR Primary and Secondary -->
-  <xacro:arg name="laser_3d_enabled"              default="$(optenv HUSKY_LASER_3D_ENABLED 0)" />
-  <xacro:arg name="laser_3d_topic"                default="$(optenv HUSKY_LASER_3D_TOPIC points)"/>
-  <xacro:arg name="laser_3d_tower"                default="$(optenv HUSKY_LASER_3D_TOWER 1)"/>
-  <xacro:arg name="laser_3d_prefix"               default="$(optenv HUSKY_LASER_3D_PREFIX )"/>
-  <xacro:arg name="laser_3d_parent"               default="$(optenv HUSKY_LASER_3D_PARENT top_plate_link)"/>
-  <xacro:arg name="laser_3d_xyz"                  default="$(optenv HUSKY_LASER_3D_XYZ 0 0 0)" />
-  <xacro:arg name="laser_3d_rpy"                  default="$(optenv HUSKY_LASER_3D_RPY 0 0 0)" />
-  <xacro:arg name="laser_3d_secondary_enabled"    default="$(optenv HUSKY_LASER_3D_SECONDARY_ENABLED 0)" />
-  <xacro:arg name="laser_3d_secondary_topic"      default="$(optenv HUSKY_LASER_3D_SECONDARY_TOPIC secondary_points)"/>
-  <xacro:arg name="laser_3d_secondary_tower"      default="$(optenv HUSKY_LASER_3D_SECONDARY_TOWER 1)"/>
-  <xacro:arg name="laser_3d_secondary_prefix"     default="$(optenv HUSKY_LASER_3D_SECONDARY_PREFIX secondary_)"/>
-  <xacro:arg name="laser_3d_secondary_parent"     default="$(optenv HUSKY_LASER_3D_SECONDARY_PARENT top_plate_link)"/>
-  <xacro:arg name="laser_3d_secondary_xyz"        default="$(optenv HUSKY_LASER_3D_SECONDARY_XYZ 0 0 0)" />
-  <xacro:arg name="laser_3d_secondary_rpy"        default="$(optenv HUSKY_LASER_3D_SECONDARY_RPY 0 0 -3.14159)" />
-  <!-- Realsense Camera Primary and Secondary -->
-  <xacro:arg name="realsense_enabled"             default="$(optenv HUSKY_REALSENSE_ENABLED 0)" />
-  <xacro:arg name="realsense_model"               default="$(optenv HUSKY_REALSENSE_MODEL d435)"/>
-  <xacro:arg name="realsense_topic"               default="$(optenv HUSKY_REALSENSE_TOPIC realsense)" />
-  <xacro:arg name="realsense_prefix"              default="$(optenv HUSKY_REALSENSE_PREFIX camera)" />
-  <xacro:arg name="realsense_parent"              default="$(optenv HUSKY_REALSENSE_PARENT top_plate_link)" />
-  <xacro:arg name="realsense_xyz"                 default="$(optenv HUSKY_REALSENSE_XYZ 0 0 0)" />
-  <xacro:arg name="realsense_rpy"                 default="$(optenv HUSKY_REALSENSE_RPY 0 0 0)" />
-  <xacro:property name="realsense_model"          value="$(arg realsense_model)"/>
-  <xacro:arg name="realsense_secondary_enabled"   default="$(optenv HUSKY_REALSENSE_SECONDARY_ENABLED 0)" />
-  <xacro:arg name="realsense_secondary_model"     default="$(optenv HUSKY_REALSENSE_SECONDARY_MODEL d435)"/>
-  <xacro:arg name="realsense_secondary_topic"     default="$(optenv HUSKY_REALSENSE_SECONDARY_TOPIC realsense_secondary)" />
-  <xacro:arg name="realsense_secondary_prefix"    default="$(optenv HUSKY_REALSENSE_SECONDARY_PREFIX camera_secondary)" />
-  <xacro:arg name="realsense_secondary_parent"    default="$(optenv HUSKY_REALSENSE_SECONDARY_PARENT top_plate_link)" />
-  <xacro:arg name="realsense_secondary_xyz"       default="$(optenv HUSKY_REALSENSE_SECONDARY_XYZ 0 0 0)" />
-  <xacro:arg name="realsense_secondary_rpy"       default="$(optenv HUSKY_REALSENSE_SECONDARY_RPY 0 0 0)" />
-  <xacro:property name="realsense_secondary_model" value="$(arg realsense_secondary_model)"/>
-  <!-- BlackflyS Camera Primary and Secondary -->
-  <xacro:arg name="blackfly_enabled"                  default="$(optenv HUSKY_BLACKFLY 0)"/>
-  <xacro:arg name="blackfly_mount_enabled"            default="$(optenv HUSKY_BLACKFLY_MOUNT_ENABLED 1)"/>
-  <xacro:arg name="blackfly_mount_angle"              default="$(optenv HUSKY_BLACKFLY_MOUNT_ANGLE 0)"/>
-  <xacro:arg name="blackfly_prefix"                   default="$(optenv HUSKY_BLACKFLY_PREFIX blackfly)"/>
-  <xacro:arg name="blackfly_parent"                   default="$(optenv HUSKY_BLACKFLY_PARENT top_plate_link)"/>
-  <xacro:arg name="blackfly_xyz"                      default="$(optenv HUSKY_BLACKFLY_XYZ 0 0 0)"/>
-  <xacro:arg name="blackfly_rpy"                      default="$(optenv HUSKY_BLACKFLY_RPY 0 0 0)"/>
-  <xacro:arg name="blackfly_secondary_enabled"        default="$(optenv HUSKY_BLACKFLY_SECONDARY 0)"/>
-  <xacro:arg name="blackfly_secondary_mount_enabled"  default="$(optenv HUSKY_BLACKFLY_SECONDARY_MOUNT_ENABLED 1)"/>
-  <xacro:arg name="blackfly_secondary_mount_angle"    default="$(optenv HUSKY_BLACKFLY_SECONDARY_MOUNT_ANGLE 0)"/>
-  <xacro:arg name="blackfly_secondary_prefix"         default="$(optenv HUSKY_BLACKFLY_SECONDARY_PREFIX blackfly_secondary)"/>
-  <xacro:arg name="blackfly_secondary_parent"         default="$(optenv HUSKY_BLACKFLY_SECONDARY_PARENT top_plate_link)"/>
-  <xacro:arg name="blackfly_secondary_xyz"            default="$(optenv HUSKY_BLACKFLY_SECONDARY_XYZ 0 0 0)"/>
-  <xacro:arg name="blackfly_secondary_rpy"            default="$(optenv HUSKY_BLACKFLY_SECONDARY_RPY 0 0 0)"/>
+  <xacro:arg name="imu_xyz"     default="$(optenv HUSKY_IMU_XYZ -0.65 0 -0.875)"/>
+  <xacro:arg name="imu_rpy"     default="$(optenv HUSKY_IMU_RPY 0 0 0)"/>
+  <xacro:arg name="imu_parent"  default="$(optenv HUSKY_IMU_PARENT sensor_arch_link)"/>
+  <!-- Ouster LiDAR -->
+  <xacro:arg name="laser_3d_parent"  default="$(optenv HUSKY_LASER_3D_PARENT sensor_arch_link)"/>
+  <xacro:arg name="laser_3d_xyz"     default="$(optenv HUSKY_LASER_3D_XYZ 0 0 2.383)" />
+  <xacro:arg name="laser_3d_rpy"     default="$(optenv HUSKY_LASER_3D_RPY 0 0 0)" />
   <!-- Bumper Extension -->
   <xacro:property name="husky_front_bumper_extend"  value="$(optenv HUSKY_FRONT_BUMPER_EXTEND 0)" />
   <xacro:property name="husky_rear_bumper_extend"   value="$(optenv HUSKY_REAR_BUMPER_EXTEND 0)" />
-  <!-- Height of the sensor arch in mm.  Must be either 510 or 300 -->
-  <xacro:arg name="sensor_arch"         default="$(optenv HUSKY_SENSOR_ARCH 0)" />
-  <xacro:arg name="sensor_arch_height"  default="$(optenv HUSKY_SENSOR_ARCH_HEIGHT 510)" />
-  <xacro:arg name="sensor_arch_xyz"     default="$(optenv HUSKY_SENSOR_ARCH_OFFSET 0 0 0)"/>
-  <xacro:arg name="sensor_arch_rpy"     default="$(optenv HUSKY_SENSOR_ARCH_RPY 0 0 0)"/>
   <!-- Extras -->
   <xacro:arg name="robot_namespace" default="$(optenv ROBOT_NAMESPACE /)" />
   <xacro:arg name="urdf_extras"     default="$(optenv HUSKY_URDF_EXTRAS empty.urdf)" />
   <xacro:arg name="cpr_urdf_extras" default="$(optenv CPR_URDF_EXTRAS empty.urdf)" />
-  <!-- OutdoorNav -->
-  <xacro:arg name="outdoornav_enabled"       default="$(optenv OUTDOORNAV_ENABLED 0)" />
-  <xacro:arg name="outdoornav_configuration" default="$(optenv OUTDOORNAV_CONFIGURATION standard)" />
   <!-- Included URDF/XACRO Files -->
-  <xacro:include filename="$(find husky_description)/urdf/accessories/hokuyo_ust10.urdf.xacro" />
-  <xacro:include filename="$(find husky_description)/urdf/accessories/intel_realsense.urdf.xacro"/>
-  <xacro:include filename="$(find husky_description)/urdf/accessories/flir_blackfly_mount.urdf.xacro"/>
-  <xacro:include filename="$(find husky_description)/urdf/accessories/sensor_arch.urdf.xacro"/>
-  <xacro:include filename="$(find husky_description)/urdf/accessories/sick_lms1xx_mount.urdf.xacro"/>
-  <xacro:include filename="$(find husky_description)/urdf/accessories/vlp16_mount.urdf.xacro"/>
   <xacro:include filename="$(find husky_description)/urdf/decorations.urdf.xacro" />
   <xacro:include filename="$(find husky_description)/urdf/wheel.urdf.xacro" />
@@ -194,16 +109,7 @@
   <xacro:husky_decorate />
   <!--
-    Add the main sensor arch if the user has specifically enabled it, or if a sensor
-    requires it for mounting
+      IMU Link: Standard location to add an IMU
   -->
-  <xacro:if value="$(arg sensor_arch)">
-    <xacro:sensor_arch prefix="" parent="top_plate_link" size="$(arg sensor_arch_height)">
-      <origin xyz="$(arg sensor_arch_xyz)" rpy="$(arg sensor_arch_rpy)"/>
-    </xacro:sensor_arch>
-  </xacro:if>
-  <!--
-      IMU Link: Standard location to add an IMU (i.e. UM7 or Microstrain)
-  -->
-  <link name="imu_link"/>
+  <link name="imu_link" />
   <joint name="imu_joint" type="fixed">
     <origin xyz="$(arg imu_xyz)" rpy="$(arg imu_rpy)" />
@@ -211,154 +117,21 @@
     <child link="imu_link" />
   </joint>
-  <gazebo reference="imu_link">
-  </gazebo>
   <!--
-    SICK LMS1XX Priamry and Secondary Laser Scans
+      Ouster Link: Standard location to add an Ouster Lidar
   -->
-  <xacro:if value="$(arg laser_enabled)">
-    <xacro:sick_lms1xx_mount prefix="$(arg laser_prefix)" parent="$(arg laser_parent)" topic="$(arg laser_topic)" robot_namespace="$(arg robot_namespace)" tower="$(arg laser_tower)">
-      <origin xyz="$(arg laser_xyz)" rpy="$(arg laser_rpy)"/>
-    </xacro:sick_lms1xx_mount>
-  </xacro:if>
-  <xacro:if value="$(arg laser_secondary_enabled)">
-    <xacro:sick_lms1xx_mount prefix="$(arg laser_secondary_prefix)" parent="$(arg laser_secondary_parent)" topic="$(arg laser_secondary_topic)" robot_namespace="$(arg robot_namespace)" tower="$(arg laser_secondary_tower)">
-      <origin xyz="$(arg laser_secondary_xyz)" rpy="$(arg laser_secondary_rpy)"/>
-    </xacro:sick_lms1xx_mount>
-  </xacro:if>
+  <link name="laser_3d_link" />
+  <joint name="laser_3d_joint" type="fixed">
+    <origin xyz="$(arg laser_3d_xyz)" rpy="$(arg laser_3d_rpy)" />
+    <parent link="$(arg laser_3d_parent)" />
+    <child link="laser_3d_link" />
+  </joint>
   <!--
-    Hokuyo UST10 Primary and Secondary Laser Scans
+      Sensor Link: Top Middle of sensor arch where cameras are mounted
   -->
-  <xacro:if value="$(arg laser_ust10_front_enabled)">
-    <xacro:hokuyo_ust10_mount topic="$(arg laser_ust10_front_topic)" prefix="$(arg laser_ust10_front_prefix)" parent_link="$(arg laser_ust10_front_parent)">
-        <origin xyz="$(arg laser_ust10_front_xyz)" rpy="$(arg laser_ust10_front_rpy)" />
-      </xacro:hokuyo_ust10_mount>
-  </xacro:if>
-  <xacro:if value="$(arg laser_ust10_rear_enabled)">
-    <xacro:hokuyo_ust10_mount topic="$(arg laser_ust10_rear_topic)" prefix="$(arg laser_ust10_rear_prefix)" parent_link="$(arg laser_ust10_rear_parent)">
-        <origin xyz="$(arg laser_ust10_rear_xyz)" rpy="$(arg laser_ust10_rear_rpy)" />
-      </xacro:hokuyo_ust10_mount>
-  </xacro:if>
-  <!-- Intel Realsense Primary and Secondary -->
-  <xacro:property name="realsense_enabled" value="$(arg realsense_enabled)"/>
-  <xacro:property name="realsense_secondary_enabled" value="$(arg realsense_secondary_enabled)"/>
-  <xacro:if value="${realsense_enabled or realsense_secondary_enabled}">
-      <xacro:if value="${realsense_model == 'd435'}">
-        <xacro:include filename="$(find realsense2_description)/urdf/_d435.urdf.xacro" />
-      </xacro:if>
-      <xacro:if value="${realsense_model == 'd435i'}">
-        <xacro:include filename="$(find realsense2_description)/urdf/_d435i.urdf.xacro" />
-      </xacro:if>
-      <xacro:if value="${realsense_model == 'd415'}">
-        <xacro:include filename="$(find realsense2_description)/urdf/_d415.urdf.xacro" />
-      </xacro:if>
-      <xacro:if value="${realsense_model == 'd455'}">
-        <xacro:include filename="$(find realsense2_description)/urdf/_d435.urdf.xacro" />
-      </xacro:if>
-  </xacro:if>
-  <xacro:if value="$(arg realsense_enabled)">
-    <xacro:realsense_sensor rs_model="$(arg realsense_model)"
-                            prefix="$(arg realsense_prefix)"
-                            parent="$(arg realsense_parent)"
-                            topic="$(arg realsense_topic)"
-                            include="0">
-      <origin xyz="$(arg realsense_xyz)" rpy="$(arg realsense_rpy)"/>
-    </xacro:realsense_sensor>
-  </xacro:if>
-  <xacro:if value="$(arg realsense_secondary_enabled)">
-    <xacro:realsense_sensor rs_model="$(arg realsense_secondary_model)"
-                            prefix="$(arg realsense_secondary_prefix)"
-                            parent="$(arg realsense_secondary_parent)"
-                            topic="$(arg realsense_secondary_topic)"
-                            include="0">
-      <origin xyz="$(arg realsense_secondary_xyz)" rpy="$(arg realsense_secondary_rpy)"/>
-    </xacro:realsense_sensor>
-  </xacro:if>
-  <!-- BlackflyS Camera Primary and Secondary -->
-  <xacro:if value="$(arg blackfly_enabled)">
-    <xacro:flir_blackfly_mount prefix="$(arg blackfly_prefix)"
-                                parent="$(arg blackfly_parent)"
-                                mount_enabled="$(arg blackfly_mount_enabled)"
-                                mount_angle="$(arg blackfly_mount_angle)">
-      <origin xyz="$(arg blackfly_xyz)" rpy="$(arg blackfly_rpy)"/>
-    </xacro:flir_blackfly_mount>
-  </xacro:if>
-  <xacro:if value="$(arg blackfly_secondary_enabled)">
-    <xacro:flir_blackfly_mount prefix="$(arg blackfly_secondary_prefix)"
-                                parent="$(arg blackfly_secondary_parent)"
-                                mount_enabled="$(arg blackfly_secondary_mount_enabled)"
-                                mount_angle="$(arg blackfly_secondary_mount_angle)">
-      <origin xyz="$(arg blackfly_secondary_xyz)" rpy="$(arg blackfly_secondary_rpy)"/>
-    </xacro:flir_blackfly_mount>
-  </xacro:if>
-  <!--
-    Velodyne 3D LiDAR Primary and Secondary
-  -->
-  <xacro:if value="$(arg laser_3d_enabled)">
-    <xacro:if value="$(arg laser_3d_tower)">
-      <xacro:vlp16_mount prefix="$(arg laser_3d_prefix)" parent_link="$(arg laser_3d_parent)" topic="$(arg laser_3d_topic)">
-        <origin xyz="$(arg laser_3d_xyz)" rpy="$(arg laser_3d_rpy)" />
-      </xacro:vlp16_mount>
-    </xacro:if>
-    <xacro:unless value="$(arg laser_3d_tower)">
-      <xacro:VLP-16 parent="$(arg laser_3d_parent)" topic="$(arg laser_3d_topic)" name="$(arg laser_3d_prefix)velodyne">
-        <origin xyz="$(arg laser_3d_xyz)" rpy="$(arg laser_3d_rpy)" />
-      </xacro:VLP-16>
-    </xacro:unless>
-  </xacro:if>
-  <xacro:if value="$(arg laser_3d_secondary_enabled)">
-    <xacro:if value="$(arg laser_3d_secondary_tower)">
-      <xacro:vlp16_mount prefix="$(arg laser_3d_secondary_prefix)" parent_link="$(arg laser_3d_secondary_parent)" topic="$(arg laser_3d_secondary_topic)">
-        <origin xyz="$(arg laser_3d_secondary_xyz)" rpy="$(arg laser_3d_secondary_rpy)" />
-      </xacro:vlp16_mount>
-    </xacro:if>
-    <xacro:unless value="$(arg laser_3d_secondary_tower)">
-      <xacro:VLP-16 parent="$(arg laser_3d_secondary_parent)" topic="$(arg laser_3d_secondary_topic)" name="$(arg laser_3d_secondary_prefix)velodyne">
-        <origin xyz="$(arg laser_3d_secondary_xyz)" rpy="$(arg laser_3d_secondary_rpy)" />
-      </xacro:VLP-16>
-    </xacro:unless>
-  </xacro:if>
-  <!-- OutdoorNav URDF Config -->
-  <xacro:if value="$(arg outdoornav_enabled)">
-    <xacro:include filename="$(find cpr_onav_description)/urdf/outdoornav_description.urdf.xacro" />
-    <xacro:outdoornav_sensors outdoornav_configuration="$(arg outdoornav_configuration)" />
-  </xacro:if>
-  <gazebo>
-    <plugin name="gazebo_ros_control" filename="libgazebo_ros_control.so">
-      <robotNamespace>$(arg robot_namespace)</robotNamespace>
-      <legacyModeNS>true</legacyModeNS>
-    </plugin>
-  </gazebo>
-  <gazebo>
-    <plugin name="imu_controller" filename="libhector_gazebo_ros_imu.so">
-      <robotNamespace>$(arg robot_namespace)</robotNamespace>
-      <updateRate>50.0</updateRate>
-      <bodyName>base_link</bodyName>
-      <topicName>imu/data</topicName>
-      <accelDrift>0.005 0.005 0.005</accelDrift>
-      <accelGaussianNoise>0.005 0.005 0.005</accelGaussianNoise>
-      <rateDrift>0.005 0.005 0.005 </rateDrift>
-      <rateGaussianNoise>0.005 0.005 0.005 </rateGaussianNoise>
-      <headingDrift>0.005</headingDrift>
-      <headingGaussianNoise>0.005</headingGaussianNoise>
-    </plugin>
-  </gazebo>
-  <gazebo>
-    <plugin name="gps_controller" filename="libhector_gazebo_ros_gps.so">
-      <robotNamespace>$(arg robot_namespace)</robotNamespace>
-      <updateRate>40</updateRate>
-      <bodyName>base_link</bodyName>
-      <frameId>base_link</frameId>
-      <topicName>navsat/fix</topicName>
-      <velocityTopicName>navsat/vel</velocityTopicName>
-      <referenceLatitude>$(optenv GAZEBO_WORLD_LAT 49.9)</referenceLatitude>
-      <referenceLongitude>$(optenv GAZEBO_WORLD_LON 8.9)</referenceLongitude>
-      <referenceHeading>90</referenceHeading>
-      <referenceAltitude>0</referenceAltitude>
-      <drift>0.0001 0.0001 0.0001</drift>
-    </plugin>
-  </gazebo>
-  <!-- Optional custom includes. -->
-  <xacro:include filename="$(arg urdf_extras)" />
-  <!-- Optional for Clearpath internal softwares -->
-  <xacro:include filename="$(arg cpr_urdf_extras)" />
+  <link name="sensor_arch_link" />
+  <joint name="sensor_arch_joint" type="fixed">
+    <origin xyz="0 0 33.642" rpy="0 0 0" />
+    <parent link="base_link" />
+    <child link="sensor_arch_link" />
+  </joint>
 </robot>

Commit message: Updated urdf

File: ros/catkin_ws/src/husky/husky_description/urdf/husky.urdf.xacro (robot description, xacro)
@@ -120,9 +120,9 @@
       Ouster Link: Standard location to add an Ouster Lidar
   -->
-  <link name="laser_3d_link" />
+  <link name="os_lidar" />
   <joint name="laser_3d_joint" type="fixed">
     <origin xyz="$(arg laser_3d_xyz)" rpy="$(arg laser_3d_rpy)" />
     <parent link="$(arg laser_3d_parent)" />
-    <child link="laser_3d_link" />
+    <child link="os_lidar" />
   </joint>
   <!--

Commit message: Updated urdf

File: ros/catkin_ws/src/husky/husky_description/urdf/husky.urdf.xacro (robot description, xacro)
@@ -23,11 +23,11 @@
 <robot name="husky" xmlns:xacro="http://ros.org/wiki/xacro">
   <!-- IMU Link -->
-  <xacro:arg name="imu_xyz"     default="$(optenv HUSKY_IMU_XYZ -0.65 0 -0.875)"/>
+  <xacro:arg name="imu_xyz"     default="$(optenv HUSKY_IMU_XYZ -0.01651 0 -0.022225)"/>
   <xacro:arg name="imu_rpy"     default="$(optenv HUSKY_IMU_RPY 0 0 0)"/>
   <xacro:arg name="imu_parent"  default="$(optenv HUSKY_IMU_PARENT sensor_arch_link)"/>
   <!-- Ouster LiDAR -->
+  <xacro:arg name="laser_3d_xyz"     default="$(optenv HUSKY_LASER_3D_XYZ 0 0 0.0605282)" />
+  <xacro:arg name="laser_3d_rpy"     default="$(optenv HUSKY_LASER_3D_RPY 0 0 0)" />
   <xacro:arg name="laser_3d_parent"  default="$(optenv HUSKY_LASER_3D_PARENT sensor_arch_link)"/>
-  <xacro:arg name="laser_3d_xyz"     default="$(optenv HUSKY_LASER_3D_XYZ 0 0 2.383)" />
-  <xacro:arg name="laser_3d_rpy"     default="$(optenv HUSKY_LASER_3D_RPY 0 0 0)" />
   <!-- Bumper Extension -->
   <xacro:property name="husky_front_bumper_extend"  value="$(optenv HUSKY_FRONT_BUMPER_EXTEND 0)" />
@@ -131,5 +131,5 @@
   <link name="sensor_arch_link" />
   <joint name="sensor_arch_joint" type="fixed">
-    <origin xyz="0 0 33.642" rpy="0 0 0" />
+    <origin xyz="0 0 0.8545068" rpy="0 0 0" />
     <parent link="base_link" />
     <child link="sensor_arch_link" />

Commit message: Updated urdf

File: ros/catkin_ws/src/husky/husky_description/urdf/husky.urdf.xacro (robot description, xacro)
@@ -120,9 +120,9 @@
       Ouster Link: Standard location to add an Ouster Lidar
   -->
-  <link name="os_lidar" />
+  <link name="os_sensor" />
   <joint name="laser_3d_joint" type="fixed">
     <origin xyz="$(arg laser_3d_xyz)" rpy="$(arg laser_3d_rpy)" />
     <parent link="$(arg laser_3d_parent)" />
-    <child link="os_lidar" />
+    <child link="os_sensor" />
   </joint>
   <!--
