Commit message: Using t265

File: ros/catkin_ws/src/husky/husky_description/urdf/husky.urdf.xacro (robot description, xacro)
@@ -23,4 +23,5 @@
 <robot name="husky" xmlns:xacro="http://ros.org/wiki/xacro">
   <!-- IMU Link -->
+  <!-- xacro:arg name="imu_xyz"     default="$(optenv HUSKY_IMU_XYZ -0.01651 0 -0.022225)"/ -->
   <xacro:arg name="imu_xyz"     default="$(optenv HUSKY_IMU_XYZ -0.01651 0 -0.022225)"/>
   <xacro:arg name="imu_rpy"     default="$(optenv HUSKY_IMU_RPY 0 0 0)"/>
@@ -118,4 +119,20 @@
   </joint>
   <!--
+      T265 Link
+  -->
+  <link name="t265_odom_frame" />
+  <link name="map" />
+  <joint name="t265_odom_joint" type="fixed">
+    <origin xyz="0 0 0" rpy="0 0 0" />
+    <parent link="map" />
+    <child link="t265_odom_frame" />
+  </joint>
+  <link name="t265_pose_frame" />
+  <joint name="t265_pose_joint" type="fixed">
+    <origin xyz="0 0 0" rpy="0 0 0" />
+    <parent link="imu_link" />
+    <child link="t265_pose_frame" />
+  </joint>
+  <!--
       Ouster Link: Standard location to add an Ouster Lidar
   -->

Commit message: Using t265

File: ros/catkin_ws/src/husky/husky_description/urdf/husky.urdf.xacro (robot description, xacro)
@@ -131,6 +131,6 @@
   <joint name="t265_pose_joint" type="fixed">
     <origin xyz="0 0 0" rpy="0 0 0" />
-    <parent link="imu_link" />
-    <child link="t265_pose_frame" />
+    <parent link="t265_pose_frame" />
+    <child link="imu_link" />
   </joint>
   <!--

Commit message: Using t265

File: ros/catkin_ws/src/husky/husky_description/urdf/husky.urdf.xacro (robot description, xacro)
@@ -121,11 +121,4 @@
       T265 Link
   -->
-  <link name="t265_odom_frame" />
-  <link name="map" />
-  <joint name="t265_odom_joint" type="fixed">
-    <origin xyz="0 0 0" rpy="0 0 0" />
-    <parent link="map" />
-    <child link="t265_odom_frame" />
-  </joint>
   <link name="t265_pose_frame" />
   <joint name="t265_pose_joint" type="fixed">

Commit message: Using t265

File: ros/catkin_ws/src/husky/husky_description/urdf/husky.urdf.xacro (robot description, xacro)
@@ -124,6 +124,6 @@
   <joint name="t265_pose_joint" type="fixed">
     <origin xyz="0 0 0" rpy="0 0 0" />
-    <parent link="t265_pose_frame" />
-    <child link="imu_link" />
+    <parent link="imu_link" />
+    <child link="t265_pose_frame" />
   </joint>
   <!--

Commit message: Adding liosam

File: ros/catkin_ws/src/husky/husky_description/urdf/husky.urdf.xacro (robot description, xacro)
@@ -111,5 +111,4 @@
   <!--
       IMU Link: Standard location to add an IMU
-  -->
   <link name="imu_link" />
   <joint name="imu_joint" type="fixed">
@@ -118,4 +117,5 @@
     <child link="imu_link" />
   </joint>
+  -->
   <!--
       T265 Link
@@ -124,5 +124,5 @@
   <joint name="t265_pose_joint" type="fixed">
     <origin xyz="0 0 0" rpy="0 0 0" />
-    <parent link="imu_link" />
+    <parent link="base_link" />
     <child link="t265_pose_frame" />
   </joint>

Commit message: Adding liosam

File: ros/catkin_ws/src/husky/husky_description/urdf/husky.urdf.xacro (robot description, xacro)
@@ -121,9 +121,9 @@
       T265 Link
   -->
-  <link name="t265_pose_frame" />
+  <link name="t265_link" />
   <joint name="t265_pose_joint" type="fixed">
-    <origin xyz="0 0 0" rpy="0 0 0" />
-    <parent link="base_link" />
-    <child link="t265_pose_frame" />
+    <origin xyz="0 -17.8 -9.65" rpy="0 0 0" />
+    <child link="base_link" />
+    <parent link="t265_link" />
   </joint>
   <!--

Commit message: Adding liosam

File: ros/catkin_ws/src/husky/husky_description/urdf/husky.urdf.xacro (robot description, xacro)
@@ -121,9 +121,9 @@
       T265 Link
   -->
-  <link name="t265_link" />
+  <link name="t265_pose_frame" />
   <joint name="t265_pose_joint" type="fixed">
-    <origin xyz="0 -17.8 -9.65" rpy="0 0 0" />
-    <child link="base_link" />
-    <parent link="t265_link" />
+    <origin xyz="0 17.8 9.65" rpy="0 0 0" />
+    <parent link="base_link" />
+    <child link="t265_pose_frame" />
   </joint>
   <!--

Commit message: Adding liosam

File: ros/catkin_ws/src/husky/husky_description/urdf/husky.urdf.xacro (robot description, xacro)
@@ -23,8 +23,8 @@
 <robot name="husky" xmlns:xacro="http://ros.org/wiki/xacro">
   <!-- IMU Link -->
-  <!-- xacro:arg name="imu_xyz"     default="$(optenv HUSKY_IMU_XYZ -0.01651 0 -0.022225)"/ -->
   <xacro:arg name="imu_xyz"     default="$(optenv HUSKY_IMU_XYZ -0.01651 0 -0.022225)"/>
+  <!--xacro:arg name="imu_xyz"     default="$(optenv HUSKY_IMU_XYZ 0 17.8 9.65)"/-->
   <xacro:arg name="imu_rpy"     default="$(optenv HUSKY_IMU_RPY 0 0 0)"/>
-  <xacro:arg name="imu_parent"  default="$(optenv HUSKY_IMU_PARENT sensor_arch_link)"/>
+  <xacro:arg name="imu_parent"  default="$(optenv HUSKY_IMU_PARENT base_link)"/>
   <!-- Ouster LiDAR -->
   <xacro:arg name="laser_3d_xyz"     default="$(optenv HUSKY_LASER_3D_XYZ 0 0 0.0605282)" />
@@ -111,4 +111,5 @@
   <!--
       IMU Link: Standard location to add an IMU
+  -->
   <link name="imu_link" />
   <joint name="imu_joint" type="fixed">
@@ -116,14 +117,4 @@
     <parent link="$(arg imu_parent)" />
     <child link="imu_link" />
-  </joint>
-  -->
-  <!--
-      T265 Link
-  -->
-  <link name="t265_pose_frame" />
-  <joint name="t265_pose_joint" type="fixed">
-    <origin xyz="0 17.8 9.65" rpy="0 0 0" />
-    <parent link="base_link" />
-    <child link="t265_pose_frame" />
   </joint>
   <!--

Commit message: Fixing IMU

File: ros/catkin_ws/src/husky/husky_description/urdf/husky.urdf.xacro (robot description, xacro)
@@ -121,10 +121,10 @@
       Ouster Link: Standard location to add an Ouster Lidar
   -->
-  <link name="os_sensor" />
+  <!--link name="os_sensor" />
   <joint name="laser_3d_joint" type="fixed">
     <origin xyz="$(arg laser_3d_xyz)" rpy="$(arg laser_3d_rpy)" />
     <parent link="$(arg laser_3d_parent)" />
     <child link="os_sensor" />
-  </joint>
+  </joint-->
   <!--
       Sensor Link: Top Middle of sensor arch where cameras are mounted

Commit message: Fixing IMU

File: ros/catkin_ws/src/husky/husky_description/urdf/husky.urdf.xacro (robot description, xacro)
@@ -121,10 +121,10 @@
       Ouster Link: Standard location to add an Ouster Lidar
   -->
-  <!--link name="os_sensor" />
+  <link name="os_sensor" />
   <joint name="laser_3d_joint" type="fixed">
     <origin xyz="$(arg laser_3d_xyz)" rpy="$(arg laser_3d_rpy)" />
     <parent link="$(arg laser_3d_parent)" />
     <child link="os_sensor" />
-  </joint-->
+  </joint>
   <!--
       Sensor Link: Top Middle of sensor arch where cameras are mounted

Commit message: mapping stuff

File: ros/catkin_ws/src/husky/husky_description/urdf/husky.urdf.xacro (robot description, xacro)
@@ -122,5 +122,5 @@
   -->
   <link name="os_sensor" />
-  <joint name="laser_3d_joint" type="fixed">
+  <joint name="os_sensor_joint" type="fixed">
     <origin xyz="$(arg laser_3d_xyz)" rpy="$(arg laser_3d_rpy)" />
     <parent link="$(arg laser_3d_parent)" />
