Commit message: Retrying liosam

File: ros/catkin_ws/src/mapping/LIO-SAM/launch/include/config/robot.urdf.xacro (robot description, xacro)
@@ -2,5 +2,11 @@
 <robot name="lio" xmlns:xacro="http://tixiaoshan.github.io/">
   <xacro:property name="PI" value="3.1415926535897931" />
+  <link name="map"></link>
   <link name="chassis_link"></link>
+  <joint name="map_joint" type="fixed">
+    <parent link="map"/>
+    <child link="base_link" />
+    <origin xyz="0 0 0" rpy="0 0 0" />
+  </joint>
   <link name="base_link"></link>
   <joint name="base_link_joint" type="fixed">
@@ -15,8 +21,8 @@
     <origin xyz="0 0 0" rpy="0 0 0" />
   </joint>
-  <link name="velodyne"> </link>
-  <joint name="velodyne_joint" type="fixed">
+  <link name="ouster"> </link>
+  <joint name="ouster_joint" type="fixed">
     <parent link="chassis_link" />
-    <child link="velodyne" />
+    <child link="ouster" />
     <origin xyz="0 0 0" rpy="0 0 0" />
   </joint>

Commit message: Retrying liosam

File: ros/catkin_ws/src/mapping/LIO-SAM/launch/include/config/robot.urdf.xacro (robot description, xacro)
@@ -21,8 +21,8 @@
     <origin xyz="0 0 0" rpy="0 0 0" />
   </joint>
-  <link name="ouster"> </link>
-  <joint name="ouster_joint" type="fixed">
+  <link name="os_sensor"> </link>
+  <joint name="os_sensor_joint" type="fixed">
     <parent link="chassis_link" />
-    <child link="ouster" />
+    <child link="os_sensor" />
     <origin xyz="0 0 0" rpy="0 0 0" />
   </joint>

Commit message: Retrying liosam

File: ros/catkin_ws/src/mapping/LIO-SAM/launch/include/config/robot.urdf.xacro (robot description, xacro)
@@ -2,11 +2,5 @@
 <robot name="lio" xmlns:xacro="http://tixiaoshan.github.io/">
   <xacro:property name="PI" value="3.1415926535897931" />
-  <link name="map"></link>
   <link name="chassis_link"></link>
-  <joint name="map_joint" type="fixed">
-    <parent link="map"/>
-    <child link="base_link" />
-    <origin xyz="0 0 0" rpy="0 0 0" />
-  </joint>
   <link name="base_link"></link>
   <joint name="base_link_joint" type="fixed">
@@ -21,8 +15,8 @@
     <origin xyz="0 0 0" rpy="0 0 0" />
   </joint>
-  <link name="os_sensor"> </link>
-  <joint name="os_sensor_joint" type="fixed">
+  <link name="velodyne"> </link>
+  <joint name="velodyne_joint" type="fixed">
     <parent link="chassis_link" />
-    <child link="os_sensor" />
+    <child link="velodyne" />
     <origin xyz="0 0 0" rpy="0 0 0" />
   </joint>

Commit message: liosam

File: ros/catkin_ws/src/mapping/LIO-SAM/launch/include/config/robot.urdf.xacro (robot description, xacro)
@@ -15,8 +15,8 @@
     <origin xyz="0 0 0" rpy="0 0 0" />
   </joint>
-  <link name="velodyne"> </link>
-  <joint name="velodyne_joint" type="fixed">
+  <link name="os_sensor"> </link>
+  <joint name="os_sensor_joint" type="fixed">
     <parent link="chassis_link" />
-    <child link="velodyne" />
+    <child link="os_sensor" />
     <origin xyz="0 0 0" rpy="0 0 0" />
   </joint>

Commit message: liosam

File: ros/catkin_ws/src/mapping/LIO-SAM/launch/include/config/robot.urdf.xacro (robot description, xacro)
@@ -21,4 +21,10 @@
     <origin xyz="0 0 0" rpy="0 0 0" />
   </joint>
+  <link name="ouster"> </link>
+  <joint name="ouster_joint" type="fixed">
+    <parent link="os_sensor" />
+    <child link="ouster" />
+    <origin xyz="0 0 0" rpy="0 0 0" />
+  </joint>
   <link name="navsat_link"> </link>
   <joint name="navsat_joint" type="fixed">

Commit message: everything broke

File: ros/catkin_ws/src/mapping/LIO-SAM/launch/include/config/robot.urdf.xacro (robot description, xacro)
@@ -9,5 +9,5 @@
     <origin xyz="0 0 0" rpy="0 0 0" />
   </joint>
-  <link name="imu_link"> </link>
+  <link name="imu_link"></link>
   <joint name="imu_joint" type="fixed">
     <parent link="chassis_link" />
@@ -15,14 +15,8 @@
     <origin xyz="0 0 0" rpy="0 0 0" />
   </joint>
-  <link name="os_sensor"> </link>
-  <joint name="os_sensor_joint" type="fixed">
+  <link name="velodyne"> </link>
+  <joint name="velodyne_joint" type="fixed">
     <parent link="chassis_link" />
-    <child link="os_sensor" />
-    <origin xyz="0 0 0" rpy="0 0 0" />
-  </joint>
-  <link name="ouster"> </link>
-  <joint name="ouster_joint" type="fixed">
-    <parent link="os_sensor" />
-    <child link="ouster" />
+    <child link="velodyne" />
     <origin xyz="0 0 0" rpy="0 0 0" />
   </joint>
